File: hardware/32u4-programmer.sch (KiCad schematic (older format))
At the start: 42 parts

Commit message: Improved EEPROM power delivery.
Parts:
- removed Q? (x2): PZT3904, Package_TO_SOT_SMD:SOT-223, symbol Transistor_BJT:PZT3904
- removed R? (x2): 1k, symbol Device:R
- added Q? (x2): PZT3904, Package_TO_SOT_SMD:SOT-223, symbol Transistor_BJT:PZT3904
- added Q? (x2): PZT3906, Package_TO_SOT_SMD:SOT-223-3_TabPin2, symbol Transistor_BJT:PZT3906
- added R? (x4): 1k, symbol Device:R
- added R? (x2): 100, symbol Device:R
- J?: symbol Connector:USB_B_Micro -> 32u4-programmer-rescue:USB_B_Micro-Connector
- J?: symbol Connector:AVR-ISP-6 -> 32u4-programmer-rescue:AVR-ISP-6-Connector
- U?: symbol MCU_Microchip_ATmega:ATmega32U4-AU -> 32u4-programmer-rescue:ATmega32U4-AU-MCU_Microchip_ATmega
- U?: symbol MCU_Microchip_ATtiny:ATtiny13A-PU -> 32u4-programmer-rescue:ATtiny13A-PU-MCU_Microchip_ATtiny
Connections:
- wire segments 281 -> 276
Other:
- moved on the sheet: C?, D?, R?, SW?
